Commit message: Fix some geometries
- Fix wheel_separation used for DiffDriveController.
-  Change the base_footprint link to be in the center of the twi wheels so the DiffDriveController can calculate the odom correctly.

File: brutusbot_description/urdf/mobile_base.xacro (robot description, xacro)
@@ -37,5 +37,5 @@
         <parent link="base_footprint"/>
         <child link="base_link" />
-        <origin xyz="0 0 ${wheel_radius + motor_height / 2.0}" rpy="0 0 0"/>
+        <origin xyz="${-motor_position} 0 ${wheel_radius + motor_height / 2.0}" rpy="0 0 0"/>
     </joint>
     <xacro:macro name="motor_link" params="prefix">
