Commit message: Add camera links to the URDF (Phase 1a)
The camera_link pose comes from config/camera_mount.yaml, relative to
base_footprint, so the extrinsic calibration (1f) can rewrite it without
touching xacro. Nominal values are hand-measured: x 0.07, z 0.21, level.
Update the plan: the level camera makes 1f use an upright checkerboard.

Co-Authored-By: Claude Opus 5.5 <noreply@anthropic.com>

File: brutusbot_description/urdf/brutusbot.xacro (robot description, xacro)
@@ -4,4 +4,5 @@
     <xacro:include filename="common_properties.xacro"/>
     <xacro:include filename="mobile_base.xacro"/>
+    <xacro:include filename="camera.xacro"/>
     <xacro:if value="$(arg is_sim)">
         <xacro:include filename="brutusbot_gazebo.xacro"/>

File: brutusbot_description/urdf/mobile_base.xacro (robot description, xacro)
@@ -16,4 +16,6 @@
     <xacro:property name="caster_wheel_mass" value="1.0" />
     <xacro:property name="caster_wheel_position" value="${(base_length / 2.0) - caster_wheel_radius - 0.005}" />
+    <xacro:property name="base_joint_x" value="${-motor_position}" />
+    <xacro:property name="base_joint_z" value="${wheel_radius + motor_height / 2.0}" />
     <link name="base_footprint"/>
     <link name="base_link">
@@ -37,5 +39,5 @@
         <parent link="base_footprint"/>
         <child link="base_link" />
-        <origin xyz="${-motor_position} 0 ${wheel_radius + motor_height / 2.0}" rpy="0 0 0"/>
+        <origin xyz="${base_joint_x} 0 ${base_joint_z}" rpy="0 0 0"/>
     </joint>
     <xacro:macro name="motor_link" params="prefix">
