Commit message: Add sim camera (Phase 1b) and fix robot geometry
Sim camera: gz camera sensor matching the C270 (640x480, 30 Hz, hfov
0.85 rad) publishing /image_raw and /camera_info, a ground-truth pose
publisher bridged to /ground_truth/pose, and worlds/empty.sdf (stock
empty world + Sensors system) as the default world.

Geometry: base 0.21 x 0.18 x 0.02, motors 0.075 long, wheels 0.03 wide
with 0.23 separation, static shafts from motors to wheels and a camera
support post. The controller wheel separation and the angular limits
derived from it (and the joystick scale) follow the new separation.

Co-Authored-By: Claude Opus 5.5 <noreply@anthropic.com>

File: brutusbot_description/urdf/brutusbot_gazebo.xacro (robot description, xacro)
@@ -27,4 +27,44 @@
         <maxVel>1.0</maxVel>
     </gazebo>
+    <!-- hfov matches the real C270 at 640x480: 2 * atan(320 / 707 px) -->
+    <gazebo reference="camera_link">
+        <sensor name="camera" type="camera">
+            <always_on>true</always_on>
+            <update_rate>30</update_rate>
+            <visualize>false</visualize>
+            <topic>image_raw</topic>
+            <gz_frame_id>camera_optical_link</gz_frame_id>
+            <camera>
+                <camera_info_topic>camera_info</camera_info_topic>
+                <horizontal_fov>0.85</horizontal_fov>
+                <image>
+                    <width>640</width>
+                    <height>480</height>
+                    <format>R8G8B8</format>
+                </image>
+                <clip>
+                    <near>0.05</near>
+                    <far>20.0</far>
+                </clip>
+                <noise>
+                    <type>gaussian</type>
+                    <mean>0.0</mean>
+                    <stddev>0.007</stddev>
+                </noise>
+            </camera>
+        </sensor>
+    </gazebo>
+    <!-- Ground-truth model pose (base_footprint in the world frame) for checking SLAM -->
+    <gazebo>
+        <plugin filename="gz-sim-pose-publisher-system" name="gz::sim::systems::PosePublisher">
+            <publish_link_pose>false</publish_link_pose>
+            <publish_sensor_pose>false</publish_sensor_pose>
+            <publish_collision_pose>false</publish_collision_pose>
+            <publish_visual_pose>false</publish_visual_pose>
+            <publish_model_pose>true</publish_model_pose>
+            <use_pose_vector_msg>false</use_pose_vector_msg>
+            <update_frequency>50</update_frequency>
+        </plugin>
+    </gazebo>
     <gazebo>
         <plugin filename="gz_ros2_control-system" name="gz_ros2_control::GazeboSimROS2ControlPlugin">

File: brutusbot_description/urdf/camera.xacro (robot description, xacro)
@@ -8,4 +8,11 @@
     <xacro:property name="camera_height" value="0.03" />
     <xacro:property name="camera_mass" value="0.05" />
+    <xacro:property name="camera_support_size" value="0.015" />
+    <xacro:property name="camera_support_mass" value="0.02" />
+    <!-- Camera pose relative to base_link (base_joint is a pure translation) -->
+    <xacro:property name="camera_x" value="${camera_mount['x'] - base_joint_x}" />
+    <xacro:property name="camera_z" value="${camera_mount['z'] - base_joint_z}" />
+    <!-- Vertical post from the top of the base to the bottom of the camera body -->
+    <xacro:property name="camera_support_height" value="${camera_z - camera_height / 2.0 - base_height}" />
     <link name="camera_link">
         <visual>
@@ -25,10 +32,32 @@
             o_xyz="${-camera_length / 2.0} 0 0" o_rpy="0 0 0"/>
     </link>
-    <!-- base_joint is a pure translation, so subtracting it gives the pose relative to base_link -->
     <joint name="camera_joint" type="fixed">
         <parent link="base_link"/>
         <child link="camera_link"/>
-        <origin xyz="${camera_mount['x'] - base_joint_x} ${camera_mount['y']} ${camera_mount['z'] - base_joint_z}"
+        <origin xyz="${camera_x} ${camera_mount['y']} ${camera_z}"
             rpy="${camera_mount['roll']} ${camera_mount['pitch']} ${camera_mount['yaw']}"/>
+    </joint>
+    <link name="camera_support_link">
+        <visual>
+            <geometry>
+                <box size="${camera_support_size} ${camera_support_size} ${camera_support_height}"/>
+            </geometry>
+            <origin xyz="0 0 ${camera_support_height / 2.0}" rpy="0 0 0"/>
+            <material name="gray"/>
+        </visual>
+        <collision>
+            <geometry>
+                <box size="${camera_support_size} ${camera_support_size} ${camera_support_height}"/>
+            </geometry>
+            <origin xyz="0 0 ${camera_support_height / 2.0}" rpy="0 0 0"/>
+        </collision>
+        <xacro:box_inertia m="${camera_support_mass}" x="${camera_support_size}" y="${camera_support_size}"
+            z="${camera_support_height}" o_xyz="0 0 ${camera_support_height / 2.0}" o_rpy="0 0 0"/>
+    </link>
+    <!-- Static, follows the nominal mount; it ignores the small roll/pitch/yaw a calibration may add -->
+    <joint name="camera_support_joint" type="fixed">
+        <parent link="base_link"/>
+        <child link="camera_support_link"/>
+        <origin xyz="${camera_x - camera_length / 2.0} ${camera_mount['y']} ${base_height}" rpy="0 0 0"/>
     </joint>
     <!-- Optical frame: z forward, x right, y down -->

File: brutusbot_description/urdf/mobile_base.xacro (robot description, xacro)
@@ -1,9 +1,9 @@
 <?xml version="1.0"?>
 <robot name="brutusbot" xmlns:xacro="http://www.ros.org/wiki/xacro">
-    <xacro:property name="base_length" value="0.3" />
-    <xacro:property name="base_width" value="0.25" />
-    <xacro:property name="base_height" value="0.1" />
+    <xacro:property name="base_length" value="0.21" />
+    <xacro:property name="base_width" value="0.18" />
+    <xacro:property name="base_height" value="0.02" />
     <xacro:property name="base_mass" value="5.0" />
-    <xacro:property name="motor_length" value="0.10" />
+    <xacro:property name="motor_length" value="0.075" />
     <xacro:property name="motor_width" value="0.056" />
     <xacro:property name="motor_height" value="0.056" />
@@ -11,5 +11,9 @@
     <xacro:property name="motor_position" value="${-((base_length / 2.0) - (motor_width / 2.0) - 0.005)}" />
     <xacro:property name="wheel_radius" value="0.05" />
-    <xacro:property name="wheel_length" value="0.02" />
+    <xacro:property name="wheel_length" value="0.03" />
+    <xacro:property name="wheel_separation" value="0.23" />
+    <!-- distance from the motor face (at the base side) to the wheel centre, along the shaft -->
+    <xacro:property name="wheel_offset" value="${wheel_separation / 2.0 - base_width / 2.0}" />
+    <xacro:property name="shaft_radius" value="0.004" />
     <xacro:property name="wheel_mass" value="1.0" />
     <xacro:property name="caster_wheel_radius" value="${(wheel_radius + motor_height / 2.0) / 2.0}" />
@@ -59,4 +63,19 @@
                 o_xyz="${-motor_length / 2.0} 0 0" o_rpy="0 0 0"/>
         </link>
+        <!-- Shaft from the motor face to the wheel centre; static, visual only -->
+        <link name="${prefix}_shaft_link">
+            <visual>
+                <geometry>
+                    <cylinder radius="${shaft_radius}" length="${wheel_offset}"/>
+                </geometry>
+                <origin xyz="${wheel_offset / 2.0} 0 0" rpy="0 ${pi / 2.0} 0"/>
+                <material name="gray"/>
+            </visual>
+        </link>
+        <joint name="${prefix}_motor_shaft_joint" type="fixed">
+            <parent link="${prefix}_motor_link"/>
+            <child link="${prefix}_shaft_link"/>
+            <origin xyz="0 0 0" rpy="0 0 0"/>
+        </joint>
     </xacro:macro>
     <xacro:motor_link prefix="left" />
@@ -96,5 +115,5 @@
         <parent link="left_motor_link"/>
         <child link="left_wheel_link"/>
-        <origin xyz="${wheel_length / 2.0} 0 0" rpy="0 ${pi / 2.0} 0"/>
+        <origin xyz="${wheel_offset} 0 0" rpy="0 ${pi / 2.0} 0"/>
         <axis xyz="0 0 1"/>
     </joint>
@@ -102,5 +121,5 @@
         <parent link="right_motor_link"/>
         <child link="right_wheel_link"/>
-        <origin xyz="${wheel_length / 2.0} 0 0" rpy="0 ${pi / 2.0} 0"/>
+        <origin xyz="${wheel_offset} 0 0" rpy="0 ${pi / 2.0} 0"/>
         <axis xyz="0 0 -1"/>
     </joint>
